File: Hardware/mug-warmer-plate.kicad_sch (KiCad schematic)
At the start: 0 parts

Commit message: Added power supply block
Parts:
- added D?: (no value), symbol Device:LED
- added J?: (no value), symbol Connector:Conn_01x02_Male
- added J?: (no value), symbol Connector:Conn_01x03_Male
- added J?: (no value), symbol Connector:USB_C_Receptacle
- added R? (x3): (no value), symbol Device:R
Connections:
- new net: J?.1 (Pin_1), J?.2 (Pin_2)
- new net: D?.2 (A), R?.2
- new net: J?.B5 (CC2), R?.1
- new net: J?.3 (Pin_3), J?.A4 (VBUS), J?.A9 (VBUS), J?.B4 (VBUS), J?.B9 (VBUS), R?.1
- new net: J?.A5 (CC1), R?.1
- new net +5V: J?.2 (Pin_2)
- new net GND: D?.1 (K), J?.1 (Pin_1), J?.A1 (GND), J?.A12 (GND), J?.B1 (GND), J?.B12 (GND), J?.S1 (SHIELD), R?.2, R?.2
Other:
- company: (none) -> KMBS Labs
- title: (none) -> Mug Warmer Plate
