File: Hardware/mug-warmer-plate.kicad_pcb (KiCad board)
At the start: 2 copper layers, 0 parts

Commit message: Initial PCB placement
Parts:
- added C1: 10nF, Capacitor_THT:C_Disc_D4.3mm_W1.9mm_P5.00mm, F.Cu at (148.6, 95.9)
- added C2: 100nF, Capacitor_THT:C_Disc_D4.3mm_W1.9mm_P5.00mm, F.Cu at (148.6, 98.4)
- added C3: 22uF, Capacitor_THT:C_Radial_D10.0mm_H12.5mm_P5.00mm, F.Cu at (149.3, 113.0)
- added C4: 1uF, Capacitor_THT:C_Radial_D10.0mm_H12.5mm_P5.00mm, F.Cu at (136.6, 132.1)
- added C5: 1nF, Capacitor_THT:C_Disc_D4.3mm_W1.9mm_P5.00mm, F.Cu at (172.1, 111.1)
- added C6: 10nF, Capacitor_THT:C_Disc_D4.3mm_W1.9mm_P5.00mm, F.Cu at (135.3, 120.7)
- added C7: 100nF, Capacitor_THT:C_Disc_D4.3mm_W1.9mm_P5.00mm, F.Cu at (135.3, 124.5)
- added C8: 22uF, Capacitor_THT:C_Radial_D10.0mm_H12.5mm_P5.00mm, F.Cu at (135.3, 113.0)
- added D1: LED, LED_THT:LED_D5.0mm, F.Cu at (124.8, 107.3)
- added D2: DIODE, Diode_THT:D_DO-41_SOD81_P7.62mm_Horizontal, F.Cu at (167.0, 106.0)
- added D3: LED, LED_THT:LED_D5.0mm, F.Cu at (138.4, 72.4)
- added D4: LED, LED_THT:LED_D5.0mm, F.Cu at (138.4, 80.0)
- added D5: LED, LED_THT:LED_D5.0mm, F.Cu at (138.4, 87.6)
- added J1: USB_C_Receptacle_USB2.0, USB_C_Power:TYPE-C-31-M-17, F.Cu at (123.5, 99.1)
- added J4: Conn_01x02_Male, Connector_PinHeader_2.54mm:PinHeader_1x04_P2.54mm_Vertical, F.Cu at (127.6, 114.9)
- added NT1: NetTie_2, NetTie:NetTie-2_SMD_Pad0.5mm, F.Cu at (176.8, 106.0)
- added Q1: IRLZ44N, Package_TO_SOT_THT:TO-220-3_Vertical, F.Cu at (162.2, 112.4)
- added R1: 5k1, Resistor_THT:R_Axial_DIN0207_L6.3mm_D2.5mm_P10.16mm_Horizontal, F.Cu at (133.0, 99.1)
- added R2: 5k1, Resistor_THT:R_Axial_DIN0207_L6.3mm_D2.5mm_P10.16mm_Horizontal, F.Cu at (133.0, 95.9)
- added R3: 1k, Resistor_THT:R_Axial_DIN0207_L6.3mm_D2.5mm_P10.16mm_Horizontal, F.Cu at (133.0, 102.2)
- added R4: 10k, Resistor_THT:R_Axial_DIN0207_L6.3mm_D2.5mm_P10.16mm_Horizontal, F.Cu at (143.2, 105.4)
- added R5: 1k, Resistor_THT:R_Axial_DIN0207_L6.3mm_D2.5mm_P10.16mm_Horizontal, F.Cu at (121.9, 81.9)
- added R6: 1k, Resistor_THT:R_Axial_DIN0207_L6.3mm_D2.5mm_P10.16mm_Horizontal, F.Cu at (121.9, 86.4)
- added R7: 1k, Resistor_THT:R_Axial_DIN0207_L6.3mm_D2.5mm_P10.16mm_Horizontal, F.Cu at (121.9, 90.8)
- added R8: 10k, Resistor_THT:R_Axial_DIN0207_L6.3mm_D2.5mm_P10.16mm_Horizontal, F.Cu at (121.9, 78.7)
- added REF**: MountingHole_2.5mm, MountingHole:MountingHole_2.5mm, F.Cu at (262.9, 134.0)
- added REF**: MountingHole_2.5mm, MountingHole:MountingHole_2.5mm, F.Cu at (184.2, 132.7)
- added REF**: MountingHole_2.5mm, MountingHole:MountingHole_2.5mm, F.Cu at (186.7, 70.5)
- added REF**: MountingHole_2.5mm, MountingHole:MountingHole_2.5mm, F.Cu at (263.5, 71.1)
- added REF**: MountingHole_2.5mm, MountingHole:MountingHole_2.5mm, F.Cu at (150.5, 104.1)
- added SW1: SW_DIP_x01, Button_Switch_THT:SW_PUSH_6mm_H4.3mm, F.Cu at (121.3, 69.8)
- added TP1: TestPoint, TestPoint:TestPoint_Pad_2.0x2.0mm, F.Cu at (123.2, 121.9)
- added TP2: TestPoint, TestPoint:TestPoint_Pad_2.0x2.0mm, F.Cu at (123.2, 114.9)
- added U1: LM35-NEB, Package_TO_SOT_THT:TO-220-3_Horizontal_TabDown, F.Cu at (158.4, 96.5)
- added U2: ATtiny85-20P, Package_DIP:DIP-8_W7.62mm, F.Cu at (130.8, 127.6)
